File: Season 1-2/Speedo/Season 2 Speedo/Season 2 Speedo.kicad_pcb (KiCad board)
At the start: 4 copper layers, 247.1 x 124.5 mm, 83 parts, among them U1 Pico

Commit message: Progress on speedo pcb
Parts:
- moved U1 18.3 mm to (245.7, 58.2)
- moved D1 1.10 mm to (36.9, 98.3)
- moved D2 1.10 mm to (42.2, 98.3)
- moved D3 1.10 mm to (47.4, 98.3)
- moved REF** 0.94 mm to (271.3, 152.8)
- moved D38 0.90 mm to (64.1, 106.2)
- moved D39 0.90 mm to (69.3, 106.2)
- moved D40 0.90 mm to (74.6, 106.2)
- moved D41 0.90 mm to (79.8, 106.2)
- moved D42 0.90 mm to (85.1, 106.2)
- moved D43 0.90 mm to (90.3, 106.2)
- moved D44 0.90 mm to (95.6, 106.2)
- moved D45 0.90 mm to (100.8, 106.2)
- moved D46 0.90 mm to (106.1, 106.2)
- moved D47 0.90 mm to (111.3, 106.2)
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Routing:
- net unconnected-(U1-GPIO6-Pad9): track 77.2 -> 92.6 mm
- net unconnected-(U1-GPIO4-Pad6): track 62.9 -> 77.8 mm
- net unconnected-(U1-GPIO5-Pad7): track 61.1 -> 68.2 mm
- net Net-(D33-DOUT): track 1.44 -> 0.00 mm
Other:
- board size 247.1 x 124.5 mm -> 248.9 x 125.7 mm

Commit message: Season 1/2 Speedo board updates
Season 1/2 Speedo board mostly complete, a few modifications still pending.
Parts:
- removed the ? at (148.1, 130.7)
- removed the ? at (239.5, 130.7)
- removed the ? at (114.2, 112.3)
- removed the ? at (114.2, 131.6)
- removed the ? at (41.0, 112.3)
- removed the ? at (41.0, 131.6)
- removed the ? at (237.0, 130.7)
- removed the ? at (237.0, 110.4)
- removed the ? at (145.5, 130.7)
- removed the ? at (145.4, 110.4)
- removed the ? at (114.2, 134.1)
- removed the ? at (41.0, 134.1)
- removed CS/SPI0 CSn: , 
- removed the Gnd at (203.2, 94.0)
- removed INTERRUPT, VCC: , 
- removed SI/SPI0 RX: , 
- removed SO/SPI0 TX: , 
- removed SPI0 SCK: , 
- added 5V: , , B.Cu at (40.4, 131.3)
- added 5V: , , B.Cu at (142.2, 82.9)
- added ?: , , F.Cu at (113.5, 131.3)
- added ?: , , F.Cu at (236.9, 109.9)
- added ?: , , F.Cu at (197.3, 82.9)
- added ?: , , F.Cu at (142.2, 65.2)
- added ?: , , F.Cu at (40.4, 113.5)
- added ?: , , F.Cu at (145.5, 130.2)
- added ?: , , F.Cu at (148.0, 130.2)
- added ?: , , F.Cu at (197.3, 65.2)
- added ?: , , F.Cu at (145.4, 109.9)
- added ?: , , F.Cu at (113.5, 133.9)
- added ?: , , F.Cu at (113.5, 113.5)
- added ?: , , F.Cu at (236.9, 130.2)
- added ?: , , F.Cu at (239.5, 130.2)
- added ?: , , F.Cu at (197.3, 85.5)
- added C1: 22pf, Capacitor_SMD:C_0805_2012Metric, B.Cu at (202.3, 105.5)
- added C2: 22pf, Capacitor_SMD:C_0805_2012Metric, B.Cu at (202.3, 100.6)
- added Gnd: , , B.Cu at (142.2, 85.5)
- added Gnd: , , B.Cu at (40.4, 133.9)
- added MCP2515: MCP2515-xSO, Package_SO:SOIC-18W_7.5x11.6mm_P1.27mm, B.Cu at (213.0, 106.3)
- added Q1: DMG2305UX, footprints:SOT91P240X110-3N_DMG2305UX-7, B.Cu at (253.6, 99.3)
- added R1: 10k, PCM_Resistor_SMD_AKL:R_0805_2012Metric_Pad1.15x1.40mm, B.Cu at (244.2, 101.5)
- added R2: 120, PCM_Resistor_SMD_AKL:R_0805_2012Metric_Pad1.15x1.40mm, B.Cu at (256.5, 107.1)
- added R3: 10k, PCM_Resistor_SMD_AKL:R_0805_2012Metric_Pad1.15x1.40mm, B.Cu at (183.3, 93.8)
- added REF**: TerminalBlock_Phoenix_MKDS-1,5-2-5.08_1x02_P5.08mm_Horizont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, TerminalBlock_Phoenix:TerminalBlock_Phoenix_MKDS-1,5-2-5.08_1x02_P5.08mm_Horizontal, B.Cu at (254.7, 129.3)
- added REF**: TerminalBlock_Phoenix_MKDS-1,5-2-5.08_1x02_P5.08mm_Horizont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, TerminalBlock_Phoenix:TerminalBlock_Phoenix_MKDS-1,5-2-5.08_1x02_P5.08mm_Horizontal, B.Cu at (254.7, 116.6)
- added TJA1050: TJA1051T, Package_SO:SOIC-8_3.9x4.9mm_P1.27mm, B.Cu at (250.1, 106.9)
- added TXB0104: TXB0104D, Package_SO:SOIC-14_3.9x8.7mm_P1.27mm, B.Cu at (183.1, 101.7)
- added Y1: 8Mhz, Crystal:Crystal_HC49-U_Vertical, B.Cu at (195.7, 99.9)
- Pico1: renamed from U1; value Pico -> Pico1
- moved Pico1 30.3 mm to (227.3, 82.3)
- moved D49 0.67 mm to (210.6, 82.1)
- moved D50 0.67 mm to (221.6, 82.1)
- moved D51 0.67 mm to (232.6, 82.1)
- moved D52 0.52 mm to (78.0, 79.1)
- moved D55 0.52 mm to (109.2, 79.1)
- moved D56 0.52 mm to (78.0, 86.4)
- moved D59 0.52 mm to (109.2, 86.4)
- moved D53 0.52 mm to (88.4, 79.1)
- moved D54 0.52 mm to (98.8, 79.1)
- moved D57 0.52 mm to (88.4, 86.4)
- moved D58 0.52 mm to (98.8, 86.4)
Connections:
- D1 pad 4: unconnected-(D1-DIN-Pad4) -> Net-(D1-DIN)
- D12 pad 1: unconnected-(D12-DOUT-Pad1) -> Net-(D12-DOUT)
- D13 pad 4: unconnected-(D13-DIN-Pad4) -> Net-(D13-DIN)
- D3 pad 1: unconnected-(D3-DOUT-Pad1) -> Net-(D3-DOUT)
- D33 pad 4: unconnected-(D33-DIN-Pad4) -> Net-(D3-DOUT)
- D4 pad 4: unconnected-(D4-DIN-Pad4) -> Net-(D4-DIN)
- D49 pad 4: unconnected-(D49-DIN-Pad4) -> Net-(D12-DOUT)
- D59 pad 2: unconnected-(D59-DOUT-Pad2) -> Net-(D4-DIN)
- D6 pad 1: unconnected-(D6-DOUT-Pad1) -> Net-(D6-DOUT)
- D7 pad 4: unconnected-(D7-DIN-Pad4) -> Net-(D6-DOUT)
- D9 pad 1: unconnected-(D9-DOUT-Pad1) -> Net-(D13-DIN)
- Pico1 pad 10: unconnected-(U1-GPIO7-Pad10) -> Net-(MCP2515-SO)
- Pico1 pad 12: unconnected-(U1-GPIO9-Pad12) -> Net-(MCP2515-~{INT})
- Pico1 pad 13: unconnected-(U1-GND-Pad13) -> GND
- Pico1 pad 18: unconnected-(U1-GND-Pad18) -> GND
- Pico1 pad 19: unconnected-(U1-GPIO14-Pad19) -> Net-(Pico1-GPIO14)
- Pico1 pad 20: unconnected-(U1-GPIO15-Pad20) -> Net-(Pico1-GPIO15)
- Pico1 pad 23: unconnected-(U1-GND-Pad23) -> GND
- Pico1 pad 28: unconnected-(U1-GND-Pad28) -> GND
- Pico1 pad 3: unconnected-(U1-GND-Pad3) -> GND
- Pico1 pad 33: unconnected-(U1-AGND-Pad33) -> GND
- Pico1 pad 36: unconnected-(U1-3V3-Pad36) -> Net-(Pico1-3V3)
- Pico1 pad 38: unconnected-(U1-GND-Pad38) -> GND
- Pico1 pad 39: unconnected-(U1-VSYS-Pad39) -> Net-(Pico1-VSYS)
- Pico1 pad 40: unconnected-(U1-VBUS-Pad40) -> Net-(Pico1-VBUS)
- Pico1 pad 6: unconnected-(U1-GPIO4-Pad6) -> Net-(MCP2515-SI)
- Pico1 pad 7: unconnected-(U1-GPIO5-Pad7) -> Net-(MCP2515-~{CS})
- Pico1 pad 8: unconnected-(U1-GND-Pad8) -> GND
- Pico1 pad 9: unconnected-(U1-GPIO6-Pad9) -> Net-(MCP2515-SCK)
- REF** pad 1: (no net) -> GND (x4)
Routing:
- net Net-(D1-DIN): track 0.00 -> 158.9 mm
- net unconnected-(D32-DOUT-Pad1): track 0.00 -> 113.3 mm
- net unconnected-(U1-GPIO6-Pad9): track 92.6 -> 0.00 mm
- net unconnected-(D10-DIN-Pad4): track 0.00 -> 86.9 mm
- net unconnected-(D48-DOUT-Pad1): track 0.00 -> 83.5 mm
- net Net-(Pico1-3V3): track 0.00 -> 80.7 mm
- net unconnected-(U1-GPIO4-Pad6): track 77.8 -> 0.00 mm
- net unconnected-(D52-DIN-Pad4): track 0.00 -> 77.0 mm
- net unconnected-(U1-GPIO5-Pad7): track 68.2 -> 0.00 mm
- net unconnected-(U1-GPIO9-Pad12): track 60.7 -> 0.00 mm
- net Net-(D12-DOUT): track 0.00 -> 59.1 mm
- net unconnected-(U1-GPIO7-Pad10): track 57.4 -> 0.00 mm
- net Net-(MCP2515-RXCAN): track 0.00 -> 53.9 mm
- net +5V: track 31.3 -> 80.8 mm, vias 11 -> 13
- net Net-(MCP2515-TXCAN): track 0.00 -> 43.8 mm
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Other:
- board text added: "5V"
- board text added: "Gnd"
- board text added: "Knight Rider® Season 1/2 Speedometer Board Made 2024 by Mark Campbell"
